File: Plate/KiCad/plate/plate.kicad_pcb (KiCad board)
At the start: 2 copper layers, 238.1 x 76.2 mm, 0 parts

Commit message: prepared files for final send to PCBWay
Parts:
- added REF**: SolderJumper-2_P1.3mm_Bridged2Bar_Pad1.0x1.5mm, Jumper:SolderJumper-2_P1.3mm_Bridged2Bar_Pad1.0x1.5mm, F.Cu at (239.7, 87.7)
- added REF**: SolderJumper-2_P1.3mm_Bridged2Bar_Pad1.0x1.5mm, Jumper:SolderJumper-2_P1.3mm_Bridged2Bar_Pad1.0x1.5mm, B.Cu at (47.0, 93.5)
Routing:
- net (no net): track 0.00 -> 223.1 mm, vias 0 -> 2
- added copper zone on B.Cu, net (none)
- added copper zone on F.Cu, net (none)
Changed lines of the file:
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@@
       (outputformat 1)
       (mirror false)
-      (drillshape 1)
+      (drillshape 0)
       (scaleselection 1)
-      (outputdirectory "")
+      (outputdirectory "Gerbers/")
     )
   )
   (net 0 "")
+  (footprint "Jumper:SolderJumper-2_P1.3mm_Bridged2Bar_Pad1.0x1.5mm" (layer "F.Cu")
+    (at 239.725 87.7)
+    (descr "SMD Solder Jumper, 1x1.5mm Pads, 0.3mm gap, bridged with 2 copper strips")
+    (tags "solder jumper open")
+    (attr exclude_from_pos_files exclude_from_bom)
+    (fp_text reference "REF**" (at 0 -1.8) (layer "F.SilkS")
+      (effects (font (size 1 1) (thickness 0.15)))
+    )
+    (fp_text value "SolderJumper-2_P1.3mm_Bridged2Bar_Pad1.0x1.5mm" (at 0 1.9) (layer "F.Fab")
+      (effects (font (size 1 1) (thickness 0.15)))
+    )
+    (fp_poly (pts (xy -0.25 -0.6)
+      (xy 0.25 -0.6)
+      (xy 0.25 -0.2)
+      (xy -0.25 -0.2)) (layer "F.Cu") (width 0) (fill solid))
+    (fp_poly (pts (xy -0.25 0.2)
+      (xy 0.25 0.2)
+      (xy 0.25 0.6)
+      (xy -0.25 0.6)) (layer "F.Cu") (width 0) (fill solid))
+    (fp_line (start -1.4 1) (end -1.4 -1) (layer "F.SilkS") (width 0.12))
+    (fp_line (start 1.4 1) (end -1.4 1) (layer "F.SilkS") (width 0.12))
+    (fp_line (start -1.4 -1) (end 1.4 -1) (layer "F.SilkS") (width 0.12))
+    (fp_line (start 1.4 -1) (end 1.4 1) (layer "F.SilkS") (width 0.12))
+    (fp_line (start -1.65 -1.25) (end -1.65 1.25) (layer "F.CrtYd") (width 0.05))
+    (fp_line (start 1.65 1.25) (end 1.65 -1.25) (layer "F.CrtYd") (width 0.05))
+    (fp_line (start -1.65 -1.25) (end 1.65 -1.25) (layer "F.CrtYd") (width 0.05))
+    (fp_line (start 1.65 1.25) (end -1.65 1.25) (layer "F.CrtYd") (width 0.05))
+    (pad "1" smd rect locked (at -0.65 0) (size 1 1.5) (layers "F.Cu" "F.Mask"))
+    (pad "2" smd rect locked (at 0.65 0) (size 1 1.5) (layers "F.Cu" "F.Mask"))
+  )
+  (footprint "Jumper:SolderJumper-2_P1.3mm_Bridged2Bar_Pad1.0x1.5mm" (layer "B.Cu")
+    (at 47 93.475 180)
+    (descr "SMD Solder Jumper, 1x1.5mm Pads, 0.3mm gap, bridged with 2 copper strips")
+    (tags "solder jumper open")
+    (attr exclude_from_pos_files exclude_from_bom)
+    (fp_text reference "REF**" (at 0 1.8) (layer "B.SilkS")
+      (effects (font (size 1 1) (thickness 0.15)) (justify mirror))
+    )
+    (fp_text value "SolderJumper-2_P1.3mm_Bridged2Bar_Pad1.0x1.5mm" (at 0 -1.9) (layer "B.Fab")
+      (effects (font (size 1 1) (thickness 0.15)) (justify mirror))
+    )
+    (fp_poly (pts (xy -0.25 -0.2)
+      (xy 0.25 -0.2)
+      (xy 0.25 -0.6)
+      (xy -0.25 -0.6)) (layer "B.Cu") (width 0) (fill solid))
+    (fp_poly (pts (xy -0.25 0.6)
+      (xy 0.25 0.6)
+      (xy 0.25 0.2)
+      (xy -0.25 0.2)) (layer "B.Cu") (width 0) (fill solid))
+    (fp_line (start -1.4 1) (end 1.4 1) (layer "B.SilkS") (width 0.12))
+    (fp_line (start 1.4 -1) (end -1.4 -1) (layer "B.SilkS") (width 0.12))
+    (fp_line (start -1.4 -1) (end -1.4 1) (layer "B.SilkS") (width 0.12))
+    (fp_line (start 1.4 1) (end 1.4 -1) (layer "B.SilkS") (width 0.12))
+    (fp_line (start 1.65 -1.25) (end 1.65 1.25) (layer "B.CrtYd") (width 0.05))
+    (fp_line (start -1.65 1.25) (end 1.65 1.25) (layer "B.CrtYd") (width 0.05))
+    (fp_line (start -1.65 1.25) (end -1.65 -1.25) (layer "B.CrtYd") (width 0.05))
+    (fp_line (start 1.65 -1.25) (end -1.65 -1.25) (layer "B.CrtYd") (width 0.05))
+    (pad "1" smd rect locked (at -0.65 0 180) (size 1 1.5) (layers "B.Cu" "B.Mask"))
+    (pad "2" smd rect locked (at 0.65 0 180) (size 1 1.5) (layers "B.Cu" "B.Mask"))
+  )
   (gr_arc (start 68.86875 116.45) (end 68.86875 116.95) (angle -90) (layer "Edge.Cuts") (width 0.25))
   (gr_arc (start 197.45625 84.4) (end 197.95625 84.4) (angle -90) (layer "Edge.Cuts") (width 0.25))
@@
   (gr_line (start 198.71875 120) (end 192.71875 120) (layer "Edge.Cuts") (width 0.25))
   (gr_line (start 236.05625 84.4) (end 236.05625 97.4) (layer "Edge.Cuts") (width 0.25))
+  (segment (start 240.375 89.775) (end 240.375 87.7) (width 0.25) (layer "F.Cu") (net 0))
+  (segment (start 239.625 90.525) (end 240.375 89.775) (width 0.25) (layer "F.Cu") (net 0))
+  (via (at 239.625 90.525) (size 0.8) (drill 0.4) (layers "F.Cu" "B.Cu") (free) (net 0))
+  (via (at 50.4 109.35) (size 0.8) (drill 0.4) (layers "F.Cu" "B.Cu") (free) (net 0))
+  (segment (start 54.45 100.2) (end 235.05 100.2) (width 0.25) (layer "B.Cu") (net 0))
+  (segment (start 50.4 109.35) (end 50.4 104.25) (width 0.25) (layer "B.Cu") (net 0))
+  (segment (start 47.65 93.475) (end 47.65 106.6) (width 0.25) (layer "B.Cu") (net 0))
+  (segment (start 239.625 95.625) (end 239.625 90.525) (width 0.25) (layer "B.Cu") (net 0))
+  (segment (start 50.4 104.25) (end 54.45 100.2) (width 0.25) (layer "B.Cu") (net 0))
+  (segment (start 235.05 100.2) (end 239.625 95.625) (width 0.25) (layer "B.Cu") (net 0))
+  (segment (start 47.65 106.6) (end 50.4 109.35) (width 0.25) (layer "B.Cu") (net 0))
+  (zone (net 0) (net_name "") (layers F&B.Cu) (hatch edge 0.508)
+    (connect_pads (clearance 0.508))
+    (min_thickness 0.254) (filled_areas_thickness no)
+    (fill yes (thermal_gap 0.508) (thermal_bridge_width 0.508))
+    (polygon
+      (pts
+        (xy 263.675 61.375)
+        (xy 263.475 139.9)
+        (xy 23.35 140.175)
+        (xy 23.2 61.25)
+      )
+    )
+  )
   (group "" (id 3635e90b-62ae-45e0-92a6-a5767f822a0f)
     (members
