File: PCB/Hotswap PCB.kicad_pcb (KiCad board)
At the start: 2 copper layers, 265.1 x 76.2 mm, 107 parts, among them J1 SSD1306_OLED, J2 JST, K1 KEYSW, K10 KEYSW, K11 KEYSW, K12 KEYSW, K13 KEYSW, K14 KEYSW, K15 KEYSW, K16 KEYSW, K17 KEYSW, K18 KEYSW, K19 KEYSW, K2 KEYSW, K20 KEYSW, K21 KEYSW, K22 KEYSW, K23 KEYSW, K24 KEYSW, K25 KEYSW, K26 KEYSW, K27 KEYSW, K28 KEYSW, K29 KEYSW, K3 KEYSW, K30 KEYSW, K31 KEYSW, K32 KEYSW, K33 KEYSW, K34 KEYSW, K35 KEYSW, K36 KEYSW, K37 KEYSW, K38 KEYSW, K39 KEYSW, K4 KEYSW, K40 KEYSW, K41 KEYSW, K42 KEYSW, K43 KEYSW, K44 KEYSW, K45 KEYSW, K46 KEYSW, K5 KEYSW, K6 KEYSW, K7 KEYSW, K8 KEYSW, K9 KEYSW, SW1 RotaryEncoder_Switch, SW2 SW_Push, U1 Elite-C, U2 nice!nano

Commit message: Added QMK Firmware, added files needed for blender renders
Parts:
- moved Acryl Mount 2.62 mm to (255.7, 133.6)
- moved Acryl Mount 2.62 mm to (255.7, 62.6)
Other:
- board text added: "+"
- board text added: "-"
Changed lines of the file:
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@@
   )
   (footprint "MountingHole:MountingHole_2.2mm_M2" (layer "F.Cu")
-    (at 253.1 133.6)
+    (at 255.725 133.6)
     (descr "Mounting Hole 2.2mm, no annular, M2")
     (tags "mounting hole 2.2mm no annular m2")
@@
   )
   (footprint "MountingHole:MountingHole_2.2mm_M2" (layer "F.Cu")
-    (at 253.1 62.6)
+    (at 255.725 62.6)
     (descr "Mounting Hole 2.2mm, no annular, M2")
     (tags "mounting hole 2.2mm no annular m2")
@@
     (pad "" thru_hole circle locked (at 6.01 2.49 90) (size 2.1 2.1) (drill 1.3) (layers *.Cu *.Mask))
     (pad "1" thru_hole circle locked (at 0 0 90) (size 1.75 1.75) (drill 0.99) (layers *.Cu *.Mask)
-      (net 58 "GND") (pinfunction "1") (pintype "passive"))
+      (net 58 "GND") (pinfunction "1"))
     (pad "2" thru_hole circle locked (at 5 0 90) (size 1.75 1.75) (drill 0.99) (layers *.Cu *.Mask)
-      (net 65 "RST") (pinfunction "2") (pintype "passive"))
+      (net 65 "RST") (pinfunction "2"))
     (model "${KISYS3DMOD}/Buttons_Switches_THT.3dshapes/SW_Tactile_SPST_Angled_PTS645Vx39-2LFS.wrl"
       (offset (xyz 0 0 0))
@@
   (gr_arc (start 98.9625 82.050001) (end 98.9625 81.550001) (angle -90) (layer "User.1") (width 0.2))
   (gr_line (start 117.5125 82.050001) (end 117.5125 95.050001) (layer "User.1") (width 0.2))
+  (gr_text "+" (at 267.6 103.775) (layer "B.SilkS")
+    (effects (font (size 1 1) (thickness 0.15)))
+  )
+  (gr_text "-" (at 267.6 101.725) (layer "B.SilkS")
+    (effects (font (size 1 1) (thickness 0.15)))
+  )
   (segment (start 30.342 64.42) (end 30.342 66.242) (width 0.25) (layer "B.Cu") (net 1))
   (segment (start 31.175 72.725) (end 28.4 75.5) (width 0.25) (layer "B.Cu") (net 1))

Commit message: prepared files for final send to PCBWay
Parts:
- added G***: LOGO, Logos:large logo, F.Cu at (191.9, 96.6)
- added G***: LOGO, Logos:Hotswap Logo, F.Cu at (36.6, 134.7)

Commit message: Removed revision naming on PCB, fixed info.json so it will now properly work, added VIA compatiblility, Updated renders slightly
Parts:
- added G***: LOGO, Logos:fine40logo, F.Cu at (140.7, 115.8)
- moved G*** 103.4 mm to (139.6, 125.1)
- moved G*** 65.4 mm to (248.3, 63.4)

Commit message: Second revision for the IC
Connections:
- D42 pad 1: row3 -> row7
Routing:
- net row7: track 133.0 -> 168.0 mm
- net row3: track 322.5 -> 318.2 mm
Changed lines of the file:
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@@
     (pad "" np_thru_hole circle locked (at 5.08 0 48.0996) (size 1.75 1.75) (drill 1.75) (layers *.Cu *.Mask))
     (pad "1" smd rect locked (at -7.085 -2.54) (size 2.55 2.5) (layers "B.Cu" "B.Paste" "B.Mask")
-      (net 63 "col4"))
+      (net 63 "col4") (pintype "passive"))
     (pad "2" smd rect locked (at 5.842 -5.08) (size 2.55 2.5) (layers "B.Cu" "B.Paste" "B.Mask")
-      (net 38 "Net-(D32-Pad2)"))
+      (net 38 "Net-(D32-Pad2)") (pintype "passive"))
     (model "${KILIB}/MX_Alps_Hybrid.pretty/MX_Only.pretty/3d_shapes/CPG151101S11.wrl"
       (offset (xyz 0 0 -1.4868))
@@
     (fp_line (start 1.778 0.762) (end 1.778 -0.762) (layer "B.SilkS") (width 0.15))
     (pad "1" smd rect locked (at 2.5 0 180) (size 2.9 0.5) (layers "B.Cu")
-      (net 44 "row3") (pinfunction "K") (pintype "passive"))
+      (net 68 "row7") (pinfunction "K") (pintype "passive"))
     (pad "1" thru_hole rect locked (at 3.9 0 180) (size 1.6 1.6) (drill 1) (layers *.Cu *.Mask "F.SilkS")
-      (net 44 "row3") (pinfunction "K") (pintype "passive"))
+      (net 68 "row7") (pinfunction "K") (pintype "passive"))
     (pad "1" smd rect locked (at 1.4 0 180) (size 1.6 1.2) (layers "B.Cu" "B.Paste" "B.Mask")
-      (net 44 "row3") (pinfunction "K") (pintype "passive"))
+      (net 68 "row7") (pinfunction "K") (pintype "passive"))
     (pad "2" smd rect locked (at -2.5 0 180) (size 2.9 0.5) (layers "B.Cu")
       (net 49 "Net-(D42-Pad2)") (pinfunction "A") (pintype "passive"))
@@
   (segment (start 83.15 135.55) (end 80.1 132.5) (width 0.25) (layer "F.Cu") (net 44))
   (segment (start 61.65 135.55) (end 42.65 135.55) (width 0.25) (layer "F.Cu") (net 44))
-  (segment (start 149.1 132.5) (end 152.15 135.55) (width 0.25) (layer "F.Cu") (net 44))
   (segment (start 176.77548 134.29952) (end 247.836197 134.29952) (width 0.25) (layer "F.Cu") (net 44))
   (segment (start 279.052011 97.289511) (end 274.2325 92.47) (width 0.25) (layer "F.Cu") (net 44))
@@
   (segment (start 239.6 132.5) (end 240.95 133.85) (width 0.25) (layer "F.Cu") (net 68))
   (segment (start 202.95 133.85) (end 181.45 133.85) (width 0.25) (layer "F.Cu") (net 68))
+  (segment (start 150.425 133.825) (end 149.1 132.5) (width 0.25) (layer "F.Cu") (net 68))
   (segment (start 222.075 133.85) (end 202.95 133.85) (width 0.25) (layer "F.Cu") (net 68))
+  (segment (start 169.15 133.85) (end 166.6 131.3) (width 0.25) (layer "F.Cu") (net 68))
+  (segment (start 166.6 131.3) (end 163.5 131.3) (width 0.25) (layer "F.Cu") (net 68))
   (segment (start 256.97 92.47) (end 254.365718 92.47) (width 0.25) (layer "F.Cu") (net 68))
   (segment (start 202.95 133.85) (end 201.6 132.5) (width 0.25) (layer "F.Cu") (net 68))
@@
   (segment (start 253.875 129.875) (end 252.47308 129.875) (width 0.25) (layer "F.Cu") (net 68))
   (segment (start 221.95 133.85) (end 220.6 132.5) (width 0.25) (layer "F.Cu") (net 68))
+  (segment (start 163.5 131.3) (end 160.975 133.825) (width 0.25) (layer "F.Cu") (net 68))
   (segment (start 181.45 133.85) (end 180.1 132.5) (width 0.25) (layer "F.Cu") (net 68))
   (segment (start 258.9925 92.47) (end 256.97 92.47) (width 0.25) (layer "F.Cu") (net 68))
+  (segment (start 160.975 133.825) (end 150.425 133.825) (width 0.25) (layer "F.Cu") (net 68))
   (segment (start 254.365718 92.47) (end 253.79904 93.036678) (width 0.25) (layer "F.Cu") (net 68))
   (segment (start 253.79904 129.79904) (end 253.875 129.875) (width 0.25) (layer "F.Cu") (net 68))
   (segment (start 252.47308 129.875) (end 251.625 129.875) (width 0.25) (layer "F.Cu") (net 68))
+  (segment (start 181.45 133.85) (end 169.15 133.85) (width 0.25) (layer "F.Cu") (net 68))
   (segment (start 254.725 129.875) (end 253.875 129.875) (width 0.25) (layer "F.Cu") (net 68))
   (segment (start 240.95 133.85) (end 222.075 133.85) (width 0.25) (layer "F.Cu") (net 68))

Commit message: Making sure all files are up to date
Parts:
- added D48: D, Keebio:Diode-Hybrid-Back, F.Cu at (274.8, 124.5)
- added D49: D, Keebio:Diode-Hybrid-Back, F.Cu at (276.8, 123.1)
Changed lines of the file:
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@@
       (drillshape 0)
       (scaleselection 1)
-      (outputdirectory "Gerber Outputs/Hotswap PCB/")
+      (outputdirectory "Gerbers/Hotswap PCB/")
     )
   )
@@
     (pad "2" smd rect locked (at -1.4 0 180) (size 1.6 1.2) (layers "B.Cu" "B.Paste" "B.Mask")
       (net 28 "Net-(D24-Pad2)") (pinfunction "A") (pintype "passive"))
+    (model "${KISYS3DMOD}/Diodes_SMD.3dshapes/D_SOD-123.step"
+      (offset (xyz 0 0 -1.8))
+      (scale (xyz 1 1 1))
+      (rotate (xyz 0 180 0))
+    )
+  )
+  (footprint "Keebio:Diode-Hybrid-Back" (layer "F.Cu")
+    (at 274.77 124.54 90)
+    (attr smd)
+    (fp_text reference "D48" (at 0.08 -1.33 90) (layer "B.SilkS")
+      (effects (font (size 0.8 0.8) (thickness 0.15)) (justify mirror))
+    )
+    (fp_text value "D" (at 0 -1.925 90) (layer "F.SilkS") hide
+      (effects (font (size 0.8 0.8) (thickness 0.15)))
+    )
+    (fp_line (start 2.413 0.762) (end 2.413 -0.762) (layer "B.SilkS") (width 0.15))
+    (fp_line (start -2.54 0.762) (end 2.54 0.762) (layer "B.SilkS") (width 0.15))
+    (fp_line (start 2.032 -0.762) (end 2.032 0.762) (layer "B.SilkS") (width 0.15))
+    (fp_line (start 2.54 -0.762) (end -2.54 -0.762) (layer "B.SilkS") (width 0.15))
+    (fp_line (start 2.159 0.762) (end 2.159 -0.762) (layer "B.SilkS") (width 0.15))
+    (fp_line (start 2.286 -0.762) (end 2.286 0.762) (layer "B.SilkS") (width 0.15))
+    (fp_line (start 1.778 0.762) (end 1.778 -0.762) (layer "B.SilkS") (width 0.15))
+    (fp_line (start 2.54 0.762) (end 2.54 -0.762) (layer "B.SilkS") (width 0.15))
+    (fp_line (start -2.54 -0.762) (end -2.54 0.762) (layer "B.SilkS") (width 0.15))
+    (fp_line (start 1.905 0.762) (end 1.905 -0.762) (layer "B.SilkS") (width 0.15))
+    (pad "1" smd rect locked (at 2.5 0 90) (size 2.9 0.5) (layers "B.Cu"))
+    (pad "1" thru_hole rect locked (at 3.9 0 90) (size 1.6 1.6) (drill 1) (layers *.Cu *.Mask "F.SilkS"))
+    (pad "1" smd rect locked (at 1.4 0 90) (size 1.6 1.2) (layers "B.Cu" "B.Paste" "B.Mask"))
+    (pad "2" smd rect locked (at -1.4 0 90) (size 1.6 1.2) (layers "B.Cu" "B.Paste" "B.Mask"))
+    (pad "2" thru_hole circle locked (at -3.9 0 90) (size 1.6 1.6) (drill 1) (layers *.Cu *.Mask "F.SilkS"))
+    (pad "2" smd rect locked (at -2.5 0 90) (size 2.9 0.5) (layers "B.Cu"))
     (model "${KISYS3DMOD}/Diodes_SMD.3dshapes/D_SOD-123.step"
       (offset (xyz 0 0 -1.8))
@@
     (model "${KISYS3DMOD}/Diodes_SMD.3dshapes/D_SOD-123.step"
       (offset (xyz 0 0 -1.8))
+      (scale (xyz 1 1 1))
+      (rotate (xyz 0 180 0))
+    )
+  )
+  (footprint "Keebio:Diode-Hybrid-Back" (layer "F.Cu")
+    (at 276.78 123.07 90)
+    (attr smd)
+    (fp_text reference "D49" (at -0.0254 1.4 90) (layer "B.SilkS")
+      (effects (font (size 0.8 0.8) (thickness 0.15)) (justify mirror))
+    )
+    (fp_text value "D" (at 0 -1.925 90) (layer "F.SilkS") hide
+      (effects (font (size 0.8 0.8) (thickness 0.15)))
+    )
+    (fp_line (start 1.905 0.762) (end 1.905 -0.762) (layer "B.SilkS") (width 0.15))
+    (fp_line (start 2.54 -0.762) (end -2.54 -0.762) (layer "B.SilkS") (width 0.15))
+    (fp_line (start 2.159 0.762) (end 2.159 -0.762) (layer "B.SilkS") (width 0.15))
+    (fp_line (start 2.286 -0.762) (end 2.286 0.762) (layer "B.SilkS") (width 0.15))
+    (fp_line (start -2.54 -0.762) (end -2.54 0.762) (layer "B.SilkS") (width 0.15))
+    (fp_line (start -2.54 0.762) (end 2.54 0.762) (layer "B.SilkS") (width 0.15))
+    (fp_line (start 1.778 0.762) (end 1.778 -0.762) (layer "B.SilkS") (width 0.15))
+    (fp_line (start 2.032 -0.762) (end 2.032 0.762) (layer "B.SilkS") (width 0.15))
+    (fp_line (start 2.54 0.762) (end 2.54 -0.762) (layer "B.SilkS") (width 0.15))
+    (fp_line (start 2.413 0.762) (end 2.413 -0.762) (layer "B.SilkS") (width 0.15))
+    (pad "1" thru_hole rect locked (at 3.9 0 90) (size 1.6 1.6) (drill 1) (layers *.Cu *.Mask "F.SilkS"))
+    (pad "1" smd rect locked (at 1.4 0 90) (size 1.6 1.2) (layers "B.Cu" "B.Paste" "B.Mask"))
+    (pad "1" smd rect locked (at 2.5 0 90) (size 2.9 0.5) (layers "B.Cu"))
+    (pad "2" thru_hole circle locked (at -3.9 0 90) (size 1.6 1.6) (drill 1) (layers *.Cu *.Mask "F.SilkS"))
+    (pad "2" smd rect locked (at -2.5 0 90) (size 2.9 0.5) (layers "B.Cu"))
+    (pad "2" smd rect locked (at -1.4 0 90) (size 1.6 1.2) (layers "B.Cu" "B.Paste" "B.Mask"))
+    (model "${KISYS3DMOD}/Diodes_SMD.3dshapes/D_SOD-123.step"
+      (offset (xyz 0 0 -1.8))
