File: PCB/PCB.kicad_pcb (KiCad board)
At the start: 2 copper layers, 265.1 x 76.2 mm, 118 parts, among them J1 SSD1306_OLED, J2 JST, K1 KEYSW, K10 KEYSW, K11 KEYSW, K12 KEYSW, K13 KEYSW, K14 KEYSW, K15 KEYSW, K16 KEYSW, K17 KEYSW, K18 KEYSW, K19 KEYSW, K2 KEYSW, K20 KEYSW, K21 KEYSW, K22 KEYSW, K23 KEYSW, K24 KEYSW, K25 KEYSW, K26 KEYSW, K27 KEYSW, K28 KEYSW, K29 KEYSW, K3 KEYSW, K30 KEYSW, K31 KEYSW, K32 KEYSW, K33 KEYSW, K34 KEYSW, K35 KEYSW, K36 KEYSW, K37 KEYSW, K38 KEYSW, K39 KEYSW, K4 KEYSW, K40 KEYSW, K41 KEYSW, K42 KEYSW, K43 KEYSW, K44 KEYSW, K45 KEYSW, K46 KEYSW, K47 KEYSW, K5 KEYSW, K6 KEYSW, K7 KEYSW, K8 KEYSW, K9 KEYSW, SW1 RotaryEncoder_Switch, SW2 SW_Push, U1 Elite-C, U2 nice!nano

Commit message: Added QMK Firmware, added files needed for blender renders
Parts:
- moved Acryl Mnt 2.62 mm to (255.7, 133.6)
- moved Acryl Mnt 2.62 mm to (255.7, 62.6)
Other:
- board text added: "+"
- board text added: "-"
Changed lines of the file:
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@@
   )
   (footprint "MountingHole:MountingHole_2.2mm_M2" (layer "F.Cu")
-    (at 253.1 133.6)
+    (at 255.725 133.6)
     (descr "Mounting Hole 2.2mm, no annular, M2")
     (tags "mounting hole 2.2mm no annular m2")
@@
   )
   (footprint "MountingHole:MountingHole_2.2mm_M2" (layer "F.Cu")
-    (at 253.1 62.6)
+    (at 255.725 62.6)
     (descr "Mounting Hole 2.2mm, no annular, M2")
     (tags "mounting hole 2.2mm no annular m2")
@@
   (gr_arc (start 98.9625 82.050001) (end 98.9625 81.550001) (angle -90) (layer "User.1") (width 0.2))
   (gr_line (start 117.5125 82.050001) (end 117.5125 95.050001) (layer "User.1") (width 0.2))
+  (gr_text "+" (at 267.5 103.75) (layer "B.SilkS")
+    (effects (font (size 1 1) (thickness 0.15)))
+  )
+  (gr_text "-" (at 267.5 101.7) (layer "B.SilkS")
+    (effects (font (size 1 1) (thickness 0.15)))
+  )
   (segment (start 34 64.5) (end 27.12 64.5) (width 0.25) (layer "F.Cu") (net 1))
   (segment (start 27.12 64.5) (end 27.04 64.42) (width 0.25) (layer "F.Cu") (net 1))

Commit message: prepared files for final send to PCBWay
Parts:
- added G***: LOGO, Logos:large logo, F.Cu at (194.6, 96.5)
- added G***: LOGO, Logos:Solder Logo, F.Cu at (35.3, 132.9)

Commit message: Removed revision naming on PCB, fixed info.json so it will now properly work, added VIA compatiblility, Updated renders slightly
Parts:
- added G***: LOGO, Logos:fine40logo, F.Cu at (142.9, 114.4)
- moved G*** 107.1 mm to (142.1, 125.6)
- moved G*** 63.2 mm to (248.3, 63.1)
